File: _electronic/mcu.kicad_sch (KiCad schematic)
At the start: 3 parts

Commit message: BETA first upload
nothing major done here:
* updated KiCAD files to v9
* removed alternative 6v feed-in. The proposed buck converter is fine.
* added to all components LCSC component IDs. With this, exporting the project as gerber files also automatically creates correct BOM for JLCPCB manufacturing
*
Parts:
- C_MCU1: LCSC (none) -> C14663
- C_MCU2: LCSC (none) -> C96446
- U_MCU1: LCSC (none) -> C473012
Other:
- title: E-TKT v1.0 -> E-TKT v2.0 BETA
