File: _electronic/power3v3.kicad_sch (KiCad schematic)
At the start: 3 parts

Commit message: BETA first upload
nothing major done here:
* updated KiCAD files to v9
* removed alternative 6v feed-in. The proposed buck converter is fine.
* added to all components LCSC component IDs. With this, exporting the project as gerber files also automatically creates correct BOM for JLCPCB manufacturing
*
Parts:
- C_POW1, C_POW2: LCSC (none) -> C96446
- U_POW2: LCSC (none) -> C92102
Other:
- title: E-TKT v1.0 -> E-TKT v2.0 BETA
