File: _electronic/e-tkt.kicad_sch (KiCad schematic)
At the start: 6 parts

Commit message: BETA first upload
nothing major done here:
* updated KiCAD files to v9
* removed alternative 6v feed-in. The proposed buck converter is fine.
* added to all components LCSC component IDs. With this, exporting the project as gerber files also automatically creates correct BOM for JLCPCB manufacturing
*
Parts:
- LS1: LCSC (none) -> C94598
Other:
- title: E-TKT v1.0 -> E-TKT v2.0 BETA

Commit message: Added CAD, cleaned up KiCAD some more
Added a FreeCAD Assembly. This will serve for minor updated to the printable parts.
Updated USB-C component to standard KiCAD libary-integrated version, because the pinout of the schematic symbol was messing with the pinout of the footprint
exported the PCB as step so it could be imported to FreeCAD
Parts:
- LS1: footprint SnapEDA Library:CUI_CSS-0575A-SMT -> EASYEDA2KICAD:BUZ-SMD_L5.0-W5.5-P4.60
Changed lines of the file:
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@@
 			)
 		)
-		(property "Footprint" "SnapEDA Library:CUI_CSS-0575A-SMT"
+		(property "Footprint" "EASYEDA2KICAD:BUZ-SMD_L5.0-W5.5-P4.60"
 			(at 143.51 104.14 0)
 			(effects
